Commit message: working bottom cabinets

File: full_pipeline_simple/initial_scene.urdf (robot description, URDF)
Before this commit: robot Scene, 13 links, 12 joints
Links:
- added link drawer_0.333_0.958_0.998_2
- added link drawer_0.333_0.958_0.998_2_corpus, mass 0.054318599999999995; collision box size=0.02 0.958 0.313; collision box size=0.02 0.958 0.313
- added link drawer_0.333_0.958_0.998_2_drawer_0_0, mass 0.1; collision box size=0.954000 0.990300 0.329000; visual mesh filename=full_pipeline_simple/drawer_0.333_0.958_0.998_2.obj
- added link drawer_0.333_0.958_0.998_3
- added link drawer_0.333_0.958_0.998_3_corpus, mass 0.054318599999999995; collision box size=0.02 0.958 0.313; collision box size=0.02 0.958 0.313
- added link drawer_0.333_0.958_0.998_3_drawer_0_0, mass 0.1; collision box size=0.954000 0.990300 0.329000; visual mesh filename=full_pipeline_simple/drawer_0.333_0.958_0.998_3.obj
- added link drawer_0.333_0.958_0.998_4
- added link drawer_0.333_0.958_0.998_4_corpus, mass 0.054318599999999995; collision box size=0.02 0.958 0.313; collision box size=0.02 0.958 0.313
- added link drawer_0.333_0.958_0.998_4_drawer_0_0, mass 0.1; collision box size=0.954000 0.990300 0.329000; visual mesh filename=full_pipeline_simple/drawer_0.333_0.958_0.998_4.obj
- added link drawer_0.333_0.958_0.998_5
- added link drawer_0.333_0.958_0.998_5_corpus, mass 0.054318599999999995; collision box size=0.02 0.958 0.313; collision box size=0.02 0.958 0.313
- added link drawer_0.333_0.958_0.998_5_drawer_0_0, mass 0.1; collision box size=0.954000 0.990300 0.329000; visual mesh filename=full_pipeline_simple/drawer_0.333_0.958_0.998_5.obj
- added link lower_left_cabinet_1.003_0.958_0.998_1
- added link lower_left_cabinet_1.003_0.958_0.998_1_corpus, mass 0.10162463999999999; collision box size=0.02 0.958 0.9829999999999999; collision box size=0.02 0.958 0.9829999999999999
- added link lower_left_cabinet_1.003_0.958_0.998_1_door_0_0, mass 0.1; collision box size=0.954000 0.168200 0.999000; visual mesh filename=full_pipeline_simple/lower_left_cabinet_1.003_0.958_0.998_1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
- added link lower_left_cabinet_1.003_0.958_0.998_2
- added link lower_left_cabinet_1.003_0.958_0.998_2_corpus, mass 0.10162463999999999; collision box size=0.02 0.958 0.9829999999999999; collision box size=0.02 0.958 0.9829999999999999
- added link lower_left_cabinet_1.003_0.958_0.998_2_door_0_0, mass 0.1; collision box size=0.954000 0.168200 0.999000; visual mesh filename=full_pipeline_simple/lower_left_cabinet_1.003_0.958_0.998_2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
- added link lower_right_cabinet_1.003_0.958_0.998_1
- added link lower_right_cabinet_1.003_0.958_0.998_1_corpus, mass 0.10162463999999999; collision box size=0.02 0.958 0.9829999999999999; collision box size=0.02 0.958 0.9829999999999999
- added link lower_right_cabinet_1.003_0.958_0.998_1_door_0_0, mass 0.1; collision box size=0.954000 0.168200 0.999000; visual mesh filename=full_pipeline_simple/lower_right_cabinet_1.003_0.958_0.998_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
- added link lower_right_cabinet_1.003_0.958_0.998_2
- added link lower_right_cabinet_1.003_0.958_0.998_2_corpus, mass 0.10162463999999999; collision box size=0.02 0.958 0.9829999999999999; collision box size=0.02 0.958 0.9829999999999999
- added link lower_right_cabinet_1.003_0.958_0.998_2_door_0_0, mass 0.1; collision box size=0.954000 0.168200 0.999000; visual mesh filename=full_pipeline_simple/lower_right_cabinet_1.003_0.958_0.998_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
Joints:
- added joint drawer_0.333_0.958_0.998_2_corpus_to_drawer_0_0: type prismatic, parent drawer_0.333_0.958_0.998_2_corpus, child drawer_0.333_0.958_0.998_2_drawer_0_0, origin xyz=0.0 -0.479 0.16649999999999998 rpy=0.0 -0.0 0.0, axis 0 -1 0, limit lower=0.0 upper=0.79218 effort=1000.0 velocity=1.0
- added joint drawer_0.333_0.958_0.998_2_origin_joint: type fixed, parent drawer_0.333_0.958_0.998_2, child drawer_0.333_0.958_0.998_2_corpus, origin xyz=0.0 0.0 0.0 rpy=0.0 -0.0 0.0
- added joint drawer_0.333_0.958_0.998_2_world_fixed_joint: type fixed, parent world, child drawer_0.333_0.958_0.998_2, origin xyz=1.916 0.0 0.0 rpy=0.0 -0.0 0.0
- added joint drawer_0.333_0.958_0.998_3_corpus_to_drawer_0_0: type prismatic, parent drawer_0.333_0.958_0.998_3_corpus, child drawer_0.333_0.958_0.998_3_drawer_0_0, origin xyz=0.0 -0.479 0.16649999999999998 rpy=0.0 -0.0 0.0, axis 0 -1 0, limit lower=0.0 upper=0.79218 effort=1000.0 velocity=1.0
- added joint drawer_0.333_0.958_0.998_3_origin_joint: type fixed, parent drawer_0.333_0.958_0.998_3, child drawer_0.333_0.958_0.998_3_corpus, origin xyz=0.0 0.0 0.0 rpy=0.0 -0.0 0.0
- added joint drawer_0.333_0.958_0.998_3_world_fixed_joint: type fixed, parent world, child drawer_0.333_0.958_0.998_3, origin xyz=2.874 0.0 0.0 rpy=0.0 -0.0 0.0
- added joint drawer_0.333_0.958_0.998_4_corpus_to_drawer_0_0: type prismatic, parent drawer_0.333_0.958_0.998_4_corpus, child drawer_0.333_0.958_0.998_4_drawer_0_0, origin xyz=0.0 -0.479 0.16649999999999998 rpy=0.0 -0.0 0.0, axis 0 -1 0, limit lower=0.0 upper=0.79218 effort=1000.0 velocity=1.0
- added joint drawer_0.333_0.958_0.998_4_origin_joint: type fixed, parent drawer_0.333_0.958_0.998_4, child drawer_0.333_0.958_0.998_4_corpus, origin xyz=0.0 0.0 0.0 rpy=0.0 -0.0 0.0
- added joint drawer_0.333_0.958_0.998_4_world_fixed_joint: type fixed, parent world, child drawer_0.333_0.958_0.998_4, origin xyz=3.8520000000000003 -0.9779999999999999 0.0 rpy=0.0 -0.0 -1.5707963267948966
- added joint drawer_0.333_0.958_0.998_5_corpus_to_drawer_0_0: type prismatic, parent drawer_0.333_0.958_0.998_5_corpus, child drawer_0.333_0.958_0.998_5_drawer_0_0, origin xyz=0.0 -0.479 0.16649999999999998 rpy=0.0 -0.0 0.0, axis 0 -1 0, limit lower=0.0 upper=0.79218 effort=1000.0 velocity=1.0
- added joint drawer_0.333_0.958_0.998_5_origin_joint: type fixed, parent drawer_0.333_0.958_0.998_5, child drawer_0.333_0.958_0.998_5_corpus, origin xyz=0.0 0.0 0.0 rpy=0.0 -0.0 0.0
- added joint drawer_0.333_0.958_0.998_5_world_fixed_joint: type fixed, parent world, child drawer_0.333_0.958_0.998_5, origin xyz=3.852 -1.936 0.0 rpy=0.0 -0.0 -1.5707963267948966
- added joint lower_left_cabinet_1.003_0.958_0.998_1_corpus_to_door_0_0: type revolute, parent lower_left_cabinet_1.003_0.958_0.998_1_corpus, child lower_left_cabinet_1.003_0.958_0.998_1_door_0_0, origin xyz=0.477 -0.499 0.5015 rpy=0.0 -0.0 0.0, axis 0 0 1, limit lower=0.0 upper=1.5707963267948966 effort=1000.0 velocity=0.1
- added joint lower_left_cabinet_1.003_0.958_0.998_1_origin_joint: type fixed, parent lower_left_cabinet_1.003_0.958_0.998_1, child lower_left_cabinet_1.003_0.958_0.998_1_corpus, origin xyz=0.0 0.0 0.0 rpy=0.0 -0.0 0.0
- added joint lower_left_cabinet_1.003_0.958_0.998_1_world_fixed_joint: type fixed, parent world, child lower_left_cabinet_1.003_0.958_0.998_1, origin xyz=2.874 0.0 -1.003 rpy=0.0 -0.0 0.0
- added joint lower_left_cabinet_1.003_0.958_0.998_2_corpus_to_door_0_0: type revolute, parent lower_left_cabinet_1.003_0.958_0.998_2_corpus, child lower_left_cabinet_1.003_0.958_0.998_2_door_0_0, origin xyz=0.477 -0.499 0.5015 rpy=0.0 -0.0 0.0, axis 0 0 1, limit lower=0.0 upper=1.5707963267948966 effort=1000.0 velocity=0.1
- added joint lower_left_cabinet_1.003_0.958_0.998_2_origin_joint: type fixed, parent lower_left_cabinet_1.003_0.958_0.998_2, child lower_left_cabinet_1.003_0.958_0.998_2_corpus, origin xyz=0.0 0.0 0.0 rpy=0.0 -0.0 0.0
- added joint lower_left_cabinet_1.003_0.958_0.998_2_world_fixed_joint: type fixed, parent world, child lower_left_cabinet_1.003_0.958_0.998_2, origin xyz=3.852 -1.936 -1.003 rpy=0.0 -0.0 -1.5707963267948966
- added joint lower_right_cabinet_1.003_0.958_0.998_1_corpus_to_door_0_0: type revolute, parent lower_right_cabinet_1.003_0.958_0.998_1_corpus, child lower_right_cabinet_1.003_0.958_0.998_1_door_0_0, origin xyz=-0.477 -0.499 0.5015 rpy=0.0 -0.0 0.0, axis 0 0 -1, limit lower=0.0 upper=1.5707963267948966 effort=1000.0 velocity=0.1
- added joint lower_right_cabinet_1.003_0.958_0.998_1_origin_joint: type fixed, parent lower_right_cabinet_1.003_0.958_0.998_1, child lower_right_cabinet_1.003_0.958_0.998_1_corpus, origin xyz=0.0 0.0 0.0 rpy=0.0 -0.0 0.0
- added joint lower_right_cabinet_1.003_0.958_0.998_1_world_fixed_joint: type fixed, parent world, child lower_right_cabinet_1.003_0.958_0.998_1, origin xyz=1.916 0.0 -1.003 rpy=0.0 -0.0 0.0
- added joint lower_right_cabinet_1.003_0.958_0.998_2_corpus_to_door_0_0: type revolute, parent lower_right_cabinet_1.003_0.958_0.998_2_corpus, child lower_right_cabinet_1.003_0.958_0.998_2_door_0_0, origin xyz=-0.477 -0.499 0.5015 rpy=0.0 -0.0 0.0, axis 0 0 -1, limit lower=0.0 upper=1.5707963267948966 effort=1000.0 velocity=0.1
- added joint lower_right_cabinet_1.003_0.958_0.998_2_origin_joint: type fixed, parent lower_right_cabinet_1.003_0.958_0.998_2, child lower_right_cabinet_1.003_0.958_0.998_2_corpus, origin xyz=0.0 0.0 0.0 rpy=0.0 -0.0 0.0
- added joint lower_right_cabinet_1.003_0.958_0.998_2_world_fixed_joint: type fixed, parent world, child lower_right_cabinet_1.003_0.958_0.998_2, origin xyz=3.852 -0.9779999999999999 -1.003 rpy=0.0 -0.0 -1.5707963267948966

Commit message: adding more geometry

File: full_pipeline_simple/initial_scene.urdf (robot description, URDF)
Before this commit: robot Scene, 37 links, 36 joints
Links:
- added link double_drawer_0.611_1.916_0.998
- added link double_drawer_0.611_1.916_0.998_corpus, mass 0.11871535999999999; collision box size=0.02 0.958 0.591; collision box size=0.02 0.958 0.591
- added link double_drawer_0.611_1.916_0.998_drawer_0_0, mass 0.10000000000000002; collision box size=1.912000 0.990300 0.607000; visual mesh filename=full_pipeline_simple/double_drawer_0.611_1.916_0.998.obj
- added link upper_left_cabinet_1.003_0.958_0.65_0
- added link upper_left_cabinet_1.003_0.958_0.65_0_corpus, mass 0.06948634; collision box size=0.01 0.62 2.0930000000000004; collision box size=0.01 0.62 2.0930000000000004
- added link upper_left_cabinet_1.003_0.958_0.65_0_door_0_0, mass 0.09999999999999998; collision box size=0.956000 0.168200 2.101000; visual mesh filename=full_pipeline_simple/upper_left_cabinet_1.003_0.958_0.65_0.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
- added link upper_left_cabinet_1.003_0.958_0.65_1
- added link upper_left_cabinet_1.003_0.958_0.65_1_corpus, mass 0.06948634; collision box size=0.01 0.62 2.0930000000000004; collision box size=0.01 0.62 2.0930000000000004
- added link upper_left_cabinet_1.003_0.958_0.65_1_door_0_0, mass 0.09999999999999998; collision box size=0.956000 0.168200 2.101000; visual mesh filename=full_pipeline_simple/upper_left_cabinet_1.003_0.958_0.65_1.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
- added link upper_left_cabinet_1.003_0.958_0.65_2
- added link upper_left_cabinet_1.003_0.958_0.65_2_corpus, mass 0.06948634; collision box size=0.01 0.62 2.0930000000000004; collision box size=0.01 0.62 2.0930000000000004
- added link upper_left_cabinet_1.003_0.958_0.65_2_door_0_0, mass 0.09999999999999998; collision box size=0.956000 0.168200 2.101000; visual mesh filename=full_pipeline_simple/upper_left_cabinet_1.003_0.958_0.65_2.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
- added link upper_left_cabinet_1.003_0.958_0.65_3
- added link upper_left_cabinet_1.003_0.958_0.65_3_corpus, mass 0.06948634; collision box size=0.01 0.62 2.0930000000000004; collision box size=0.01 0.62 2.0930000000000004
- added link upper_left_cabinet_1.003_0.958_0.65_3_door_0_0, mass 0.09999999999999998; collision box size=0.956000 0.168200 2.101000; visual mesh filename=full_pipeline_simple/upper_left_cabinet_1.003_0.958_0.65_3.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
- added link upper_right_cabinet_1.003_0.958_0.65_0
- added link upper_right_cabinet_1.003_0.958_0.65_0_corpus, mass 0.06948634; collision box size=0.01 0.62 2.0930000000000004; collision box size=0.01 0.62 2.0930000000000004
- added link upper_right_cabinet_1.003_0.958_0.65_0_door_0_0, mass 0.09999999999999998; collision box size=0.956000 0.168200 2.101000; visual mesh filename=full_pipeline_simple/upper_right_cabinet_1.003_0.958_0.65_0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
- added link upper_right_cabinet_1.003_0.958_0.65_1
- added link upper_right_cabinet_1.003_0.958_0.65_1_corpus, mass 0.06948634; collision box size=0.01 0.62 2.0930000000000004; collision box size=0.01 0.62 2.0930000000000004
- added link upper_right_cabinet_1.003_0.958_0.65_1_door_0_0, mass 0.09999999999999998; collision box size=0.956000 0.168200 2.101000; visual mesh filename=full_pipeline_simple/upper_right_cabinet_1.003_0.958_0.65_1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
- added link upper_right_cabinet_1.003_0.958_0.65_2
- added link upper_right_cabinet_1.003_0.958_0.65_2_corpus, mass 0.06948634; collision box size=0.01 0.62 2.0930000000000004; collision box size=0.01 0.62 2.0930000000000004
- added link upper_right_cabinet_1.003_0.958_0.65_2_door_0_0, mass 0.09999999999999998; collision box size=0.956000 0.168200 2.101000; visual mesh filename=full_pipeline_simple/upper_right_cabinet_1.003_0.958_0.65_2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
- added link upper_right_cabinet_1.003_0.958_0.65_3
- added link upper_right_cabinet_1.003_0.958_0.65_3_corpus, mass 0.06948634; collision box size=0.01 0.62 2.0930000000000004; collision box size=0.01 0.62 2.0930000000000004
- added link upper_right_cabinet_1.003_0.958_0.65_3_door_0_0, mass 0.09999999999999998; collision box size=0.956000 0.168200 2.101000; visual mesh filename=full_pipeline_simple/upper_right_cabinet_1.003_0.958_0.65_3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
Joints:
- added joint double_drawer_0.611_1.916_0.998_corpus_to_drawer_0_0: type prismatic, parent double_drawer_0.611_1.916_0.998_corpus, child double_drawer_0.611_1.916_0.998_drawer_0_0, origin xyz=0.0 -0.479 0.3055 rpy=0.0 -0.0 0.0, axis 0 -1 0, limit lower=0.0 upper=0.79218 effort=1000.0 velocity=1.0
- added joint double_drawer_0.611_1.916_0.998_origin_joint: type fixed, parent double_drawer_0.611_1.916_0.998, child double_drawer_0.611_1.916_0.998_corpus, origin xyz=0.0 0.0 0.0 rpy=0.0 -0.0 0.0
- added joint double_drawer_0.611_1.916_0.998_world_fixed_joint: type fixed, parent world, child double_drawer_0.611_1.916_0.998, origin xyz=-1.4369999999999998 0.0 -1.003 rpy=0.0 -0.0 0.0
- added joint upper_left_cabinet_1.003_0.958_0.65_0_corpus_to_door_0_0: type revolute, parent upper_left_cabinet_1.003_0.958_0.65_0_corpus, child upper_left_cabinet_1.003_0.958_0.65_0_door_0_0, origin xyz=0.478 -0.325 1.0515000000000003 rpy=0.0 -0.0 0.0, axis 0 0 1, limit lower=0.0 upper=1.5707963267948966 effort=1000.0 velocity=0.1
- added joint upper_left_cabinet_1.003_0.958_0.65_0_origin_joint: type fixed, parent upper_left_cabinet_1.003_0.958_0.65_0, child upper_left_cabinet_1.003_0.958_0.65_0_corpus, origin xyz=0.0 0.0 0.0 rpy=0.0 -0.0 0.0
- added joint upper_left_cabinet_1.003_0.958_0.65_0_world_fixed_joint: type fixed, parent world, child upper_left_cabinet_1.003_0.958_0.65_0, origin xyz=2.874 0.174 1.233 rpy=0.0 -0.0 0.0
- added joint upper_left_cabinet_1.003_0.958_0.65_1_corpus_to_door_0_0: type revolute, parent upper_left_cabinet_1.003_0.958_0.65_1_corpus, child upper_left_cabinet_1.003_0.958_0.65_1_door_0_0, origin xyz=0.478 -0.325 1.0515000000000003 rpy=0.0 -0.0 0.0, axis 0 0 1, limit lower=0.0 upper=1.5707963267948966 effort=1000.0 velocity=0.1
- added joint upper_left_cabinet_1.003_0.958_0.65_1_origin_joint: type fixed, parent upper_left_cabinet_1.003_0.958_0.65_1, child upper_left_cabinet_1.003_0.958_0.65_1_corpus, origin xyz=0.0 0.0 0.0 rpy=0.0 -0.0 0.0
- added joint upper_left_cabinet_1.003_0.958_0.65_1_world_fixed_joint: type fixed, parent world, child upper_left_cabinet_1.003_0.958_0.65_1, origin xyz=0.9579999999999999 0.174 1.2330000000000003 rpy=0.0 -0.0 0.0
- added joint upper_left_cabinet_1.003_0.958_0.65_2_corpus_to_door_0_0: type revolute, parent upper_left_cabinet_1.003_0.958_0.65_2_corpus, child upper_left_cabinet_1.003_0.958_0.65_2_door_0_0, origin xyz=0.478 -0.325 1.0515000000000003 rpy=0.0 -0.0 0.0, axis 0 0 1, limit lower=0.0 upper=1.5707963267948966 effort=1000.0 velocity=0.1
- added joint upper_left_cabinet_1.003_0.958_0.65_2_origin_joint: type fixed, parent upper_left_cabinet_1.003_0.958_0.65_2, child upper_left_cabinet_1.003_0.958_0.65_2_corpus, origin xyz=0.0 0.0 0.0 rpy=0.0 -0.0 0.0
- added joint upper_left_cabinet_1.003_0.958_0.65_2_world_fixed_joint: type fixed, parent world, child upper_left_cabinet_1.003_0.958_0.65_2, origin xyz=-0.9580000000000001 0.174 1.2330000000000003 rpy=0.0 -0.0 0.0
- added joint upper_left_cabinet_1.003_0.958_0.65_3_corpus_to_door_0_0: type revolute, parent upper_left_cabinet_1.003_0.958_0.65_3_corpus, child upper_left_cabinet_1.003_0.958_0.65_3_door_0_0, origin xyz=0.478 -0.325 1.0515000000000003 rpy=0.0 -0.0 0.0, axis 0 0 1, limit lower=0.0 upper=1.5707963267948966 effort=1000.0 velocity=0.1
- added joint upper_left_cabinet_1.003_0.958_0.65_3_origin_joint: type fixed, parent upper_left_cabinet_1.003_0.958_0.65_3, child upper_left_cabinet_1.003_0.958_0.65_3_corpus, origin xyz=0.0 0.0 0.0 rpy=0.0 -0.0 0.0
- added joint upper_left_cabinet_1.003_0.958_0.65_3_world_fixed_joint: type fixed, parent world, child upper_left_cabinet_1.003_0.958_0.65_3, origin xyz=4.026 -1.936 1.233 rpy=0.0 -0.0 -1.5707963267948966
- added joint upper_right_cabinet_1.003_0.958_0.65_0_corpus_to_door_0_0: type revolute, parent upper_right_cabinet_1.003_0.958_0.65_0_corpus, child upper_right_cabinet_1.003_0.958_0.65_0_door_0_0, origin xyz=-0.478 -0.325 1.0515000000000003 rpy=0.0 -0.0 0.0, axis 0 0 -1, limit lower=0.0 upper=1.5707963267948966 effort=1000.0 velocity=0.1
- added joint upper_right_cabinet_1.003_0.958_0.65_0_origin_joint: type fixed, parent upper_right_cabinet_1.003_0.958_0.65_0, child upper_right_cabinet_1.003_0.958_0.65_0_corpus, origin xyz=0.0 0.0 0.0 rpy=0.0 -0.0 0.0
- added joint upper_right_cabinet_1.003_0.958_0.65_0_world_fixed_joint: type fixed, parent world, child upper_right_cabinet_1.003_0.958_0.65_0, origin xyz=1.916 0.174 1.2330000000000003 rpy=0.0 -0.0 0.0
- added joint upper_right_cabinet_1.003_0.958_0.65_1_corpus_to_door_0_0: type revolute, parent upper_right_cabinet_1.003_0.958_0.65_1_corpus, child upper_right_cabinet_1.003_0.958_0.65_1_door_0_0, origin xyz=-0.478 -0.325 1.0515000000000003 rpy=0.0 -0.0 0.0, axis 0 0 -1, limit lower=0.0 upper=1.5707963267948966 effort=1000.0 velocity=0.1
- added joint upper_right_cabinet_1.003_0.958_0.65_1_origin_joint: type fixed, parent upper_right_cabinet_1.003_0.958_0.65_1, child upper_right_cabinet_1.003_0.958_0.65_1_corpus, origin xyz=0.0 0.0 0.0 rpy=0.0 -0.0 0.0
- added joint upper_right_cabinet_1.003_0.958_0.65_1_world_fixed_joint: type fixed, parent world, child upper_right_cabinet_1.003_0.958_0.65_1, origin xyz=-1.1102230246251565e-16 0.174 1.2330000000000003 rpy=0.0 -0.0 0.0
- added joint upper_right_cabinet_1.003_0.958_0.65_2_corpus_to_door_0_0: type revolute, parent upper_right_cabinet_1.003_0.958_0.65_2_corpus, child upper_right_cabinet_1.003_0.958_0.65_2_door_0_0, origin xyz=-0.478 -0.325 1.0515000000000003 rpy=0.0 -0.0 0.0, axis 0 0 -1, limit lower=0.0 upper=1.5707963267948966 effort=1000.0 velocity=0.1
- added joint upper_right_cabinet_1.003_0.958_0.65_2_origin_joint: type fixed, parent upper_right_cabinet_1.003_0.958_0.65_2, child upper_right_cabinet_1.003_0.958_0.65_2_corpus, origin xyz=0.0 0.0 0.0 rpy=0.0 -0.0 0.0
- added joint upper_right_cabinet_1.003_0.958_0.65_2_world_fixed_joint: type fixed, parent world, child upper_right_cabinet_1.003_0.958_0.65_2, origin xyz=-1.916 0.174 1.2330000000000003 rpy=0.0 -0.0 0.0
- added joint upper_right_cabinet_1.003_0.958_0.65_3_corpus_to_door_0_0: type revolute, parent upper_right_cabinet_1.003_0.958_0.65_3_corpus, child upper_right_cabinet_1.003_0.958_0.65_3_door_0_0, origin xyz=-0.478 -0.325 1.0515000000000003 rpy=0.0 -0.0 0.0, axis 0 0 -1, limit lower=0.0 upper=1.5707963267948966 effort=1000.0 velocity=0.1
- added joint upper_right_cabinet_1.003_0.958_0.65_3_origin_joint: type fixed, parent upper_right_cabinet_1.003_0.958_0.65_3, child upper_right_cabinet_1.003_0.958_0.65_3_corpus, origin xyz=0.0 0.0 0.0 rpy=0.0 -0.0 0.0
- added joint upper_right_cabinet_1.003_0.958_0.65_3_world_fixed_joint: type fixed, parent world, child upper_right_cabinet_1.003_0.958_0.65_3, origin xyz=4.026 -0.9779999999999999 1.2330000000000003 rpy=0.0 -0.0 -1.5707963267948966

Commit message: working, trying to fix door alignment

File: full_pipeline_simple/initial_scene.urdf (robot description, URDF)
Before this commit: robot Scene, 64 links, 63 joints
Links:
- added link titled_upper_right_cabinet_2.103_0.4921463197058371_0.9192388155425117_0
- added link titled_upper_right_cabinet_2.103_0.4921463197058371_0.9192388155425117_0_corpus, mass 0.0645452550490508; collision box size=0.01 0.8892388155425117 2.0930000000000004; collision box size=0.01 0.8892388155425117 2.0930000000000004
- added link titled_upper_right_cabinet_2.103_0.4921463197058371_0.9192388155425117_0_door_0_0, mass 0.09999999999999999; collision box size=0.490146 0.168200 2.101000; visual mesh filename=full_pipeline_simple/titled_upper_right_cabinet_2.103_0.492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
Joints:
- added joint titled_upper_right_cabinet_2.103_0.4921463197058371_0.9192388155425117_0_corpus_to_door_0_0: type revolute, parent titled_upper_right_cabinet_2.103_0.4921463197058371_0.9192388155425117_0_corpus, child titled_upper_right_cabinet_2.103_0.4921463197058371_0.9192388155425117_0_door_0_0, origin xyz=-0.24507315985291855 -0.4596194077712559 1.0515000000000003 rpy=0.0 -0.0 0.0, axis 0 0 -1, limit lower=0.0 upper=1.5707963267948966 effort=1000.0 velocity=0.1
- added joint titled_upper_right_cabinet_2.103_0.4921463197058371_0.9192388155425117_0_origin_joint: type fixed, parent titled_upper_right_cabinet_2.103_0.4921463197058371_0.9192388155425117_0, child titled_upper_right_cabinet_2.103_0.4921463197058371_0.9192388155425117_0_corpus, origin xyz=0.0 0.0 0.0 rpy=0.0 -0.0 0.0
- added joint titled_upper_right_cabinet_2.103_0.4921463197058371_0.9192388155425117_0_world_fixed_joint: type fixed, parent world, child titled_upper_right_cabinet_2.103_0.4921463197058371_0.9192388155425117_0, origin xyz=3.8520000000000003 0.0 1.2330000000000003 rpy=0.0 -0.0 -0.7853981633974482
