Commit message: basement kitchen fully complete

File: basement_kitchen_pipleine/basement_kitchen.urdf (robot description, URDF)
Before this commit: robot Scene, 67 links, 66 joints
Links:
- added link counter_0, mass 0.34049238299999995; collision box size=4.938 1.04475 0.06599999999999999; visual box size=4.938 1.04475 0.06599999999999999
- added link counter_1, mass 0.18210619349999999; collision box size=2.641 1.04475 0.06599999999999999; visual box size=2.641 1.04475 0.06599999999999999
- added link microwave
- added link microwave_corpus, mass 0.13214763599999999; collision box size=0.04 0.6165 0.5164999999999998; collision box size=0.12 0.6565 0.5564999999999999
- added link microwave_door, mass 0.023305316666928706; collision box size=1.0322 0.04 0.5564999999999999; collision mesh filename=microwave_door_handle.obj
- added link refrigerator
- added link refrigerator_corpus, mass 1.0099313199999995; collision box size=0.07 0.855 2.836; collision box size=0.07 0.855 2.836
- added link refrigerator_door, mass 0.22823973989662763; collision box size=0.01 0.1 0.01; collision box size=0.01 0.1 0.01
- added link refrigerator_freezer_door, mass 0.04455075938393452; collision mesh filename=refrigerator_freezer_door_handle.obj; collision mesh filename=refrigerator_freezer_door_panel.obj
Joints:
- added joint counter_0_world_fixed_joint: type fixed, parent world, child counter_0, origin xyz=0.41150000000000064 -0.024875000000000036 0.352 rpy=0.0 -0.0 0.0
- added joint counter_1_world_fixed_joint: type fixed, parent world, child counter_1, origin xyz=3.3531249999999995 -0.8229999999999995 0.352 rpy=0.0 -0.0 -1.5707963267948966
- added joint microwave_door_joint: type revolute, parent microwave_corpus, child microwave_door, origin xyz=-0.5761 -0.30825 0.0 rpy=0.0 -0.0 0.0, axis -0.0 -0.0 -1.0, limit lower=0 upper=3.141592653589793 effort=100.0 velocity=100.0
- added joint microwave_origin_joint: type fixed, parent microwave, child microwave_corpus, origin xyz=0.0 0.0 0.0 rpy=0.0 -0.0 0.0
- added joint microwave_world_fixed_joint: type fixed, parent world, child microwave, origin xyz=-1.2345000000000002 0.020656720000000017 -0.47599999999999987 rpy=0.0 -0.0 0.0
- added joint refrigerator_door_joint: type revolute, parent refrigerator_corpus, child refrigerator_door, origin xyz=0.823 -0.4275 0.0 rpy=0.0 -0.0 0.0, axis 0.0 0.0 1.0, limit lower=0 upper=3.141592653589793 effort=100.0 velocity=100.0
- added joint refrigerator_freezer_door_joint: type revolute, parent refrigerator_corpus, child refrigerator_freezer_door, origin xyz=0.823 -0.4275 0.0 rpy=0.0 -0.0 0.0, axis 0.0 0.0 1.0, limit lower=0 upper=3.141592653589793 effort=100.0 velocity=100.0
- added joint refrigerator_origin_joint: type fixed, parent refrigerator, child refrigerator_corpus, origin xyz=0.0 0.0 0.0 rpy=0.0 -0.0 0.0
- added joint refrigerator_world_fixed_joint: type fixed, parent world, child refrigerator, origin xyz=-2.8805 -5.551115123125783e-17 -1.001 rpy=0.0 -0.0 0.0
