Commit message: final scene minus extra assests

File: initial_scene/initial_scene_2.urdf (robot description, URDF)
Before this commit: robot Scene, 67 links, 66 joints
Links:
- added link counter_0, mass 0.40235839056000006; collision box size=5.747999999999999 1.0479 0.0668; visual box size=5.747999999999999 1.0479 0.0668
- added link counter_1, mass 0.20397918407999996; collision box size=2.9139999999999997 1.0479 0.0668; visual box size=2.9139999999999997 1.0479 0.0668
- added link microwave
- added link microwave_corpus, mass 0.15063484879999997; collision box size=0.04 0.6186 0.5455499999999998; collision box size=0.12 0.6586 0.5855499999999998
- added link microwave_door, mass 0.02894979471300859; collision box size=1.2212 0.04 0.5855499999999998; collision mesh filename=microwave_door_handle.obj
- added link refrigerator
- added link refrigerator_corpus, mass 1.2616414400000002; collision box size=0.07 0.858 3.369; collision box size=0.07 0.858 3.369
- added link refrigerator_door, mass 0.32377237550989996; collision box size=0.01 0.1 0.01; collision box size=0.01 0.1 0.01
- added link refrigerator_freezer_door, mass 0.051806285527331804; collision mesh filename=refrigerator_freezer_door_handle.obj; collision mesh filename=refrigerator_freezer_door_panel.obj
Joints:
- added joint counter_0_world_fixed_joint: type fixed, parent world, child counter_0, origin xyz=0.47900000000000054 -0.024950000000000028 0.3664 rpy=0.0 -0.0 0.0
- added joint counter_1_world_fixed_joint: type fixed, parent world, child counter_1, origin xyz=3.82705 -0.9580000000000002 0.3664 rpy=0.0 -0.0 -1.5707963267948966
- added joint microwave_door_joint: type revolute, parent microwave_corpus, child microwave_door, origin xyz=-0.6706 -0.3093 0.0 rpy=0.0 -0.0 0.0, axis -0.0 -0.0 -1.0, limit lower=0 upper=3.141592653589793 effort=100.0 velocity=100.0
- added joint microwave_origin_joint: type fixed, parent microwave, child microwave_corpus, origin xyz=0.0 0.0 0.0 rpy=0.0 -0.0 0.0
- added joint microwave_world_fixed_joint: type fixed, parent world, child microwave, origin xyz=-1.4369999999999998 0.02065165999999999 -0.5034999999999998 rpy=0.0 -0.0 0.0
- added joint refrigerator_door_joint: type revolute, parent refrigerator_corpus, child refrigerator_door, origin xyz=0.958 -0.429 0.0 rpy=0.0 -0.0 0.0, axis 0.0 0.0 1.0, limit lower=0 upper=3.141592653589793 effort=100.0 velocity=100.0
- added joint refrigerator_freezer_door_joint: type revolute, parent refrigerator_corpus, child refrigerator_freezer_door, origin xyz=0.958 -0.429 0.0 rpy=0.0 -0.0 0.0, axis 0.0 0.0 1.0, limit lower=0 upper=3.141592653589793 effort=100.0 velocity=100.0
- added joint refrigerator_origin_joint: type fixed, parent refrigerator, child refrigerator_corpus, origin xyz=0.0 0.0 0.0 rpy=0.0 -0.0 0.0
- added joint refrigerator_world_fixed_joint: type fixed, parent world, child refrigerator, origin xyz=-3.3529999999999998 0.0 -1.003 rpy=0.0 -0.0 0.0
