Commit message: second floor done

File: initial_scene/initial_scene_2.urdf (robot description, URDF)
Before this commit: robot Scene, 76 links, 75 joints
Links:
- removed link double_drawer_0.49950000000000006_1.916_0.998
- removed link double_drawer_0.49950000000000006_1.916_0.998_corpus
- removed link double_drawer_0.49950000000000006_1.916_0.998_drawer_0_0
- removed link lower_left_cabinet_1.003_0.958_0.998_0
- removed link lower_left_cabinet_1.003_0.958_0.998_0_corpus
- removed link lower_left_cabinet_1.003_0.958_0.998_0_door_0_0
- removed link lower_left_cabinet_1.003_0.958_0.998_1
- removed link lower_left_cabinet_1.003_0.958_0.998_1_corpus
- removed link lower_left_cabinet_1.003_0.958_0.998_1_door_0_0
- removed link lower_left_cabinet_1.003_0.958_0.998_2
- removed link lower_left_cabinet_1.003_0.958_0.998_2_corpus
- removed link lower_left_cabinet_1.003_0.958_0.998_2_door_0_0
- removed link titled_upper_right_cabinet_2.103_0.7056925676241745_0.7056925676241744_0
- removed link titled_upper_right_cabinet_2.103_0.7056925676241745_0.7056925676241744_0_corpus
- removed link titled_upper_right_cabinet_2.103_0.7056925676241745_0.7056925676241744_0_door_0_0
- removed link upper_left_cabinet_1.003_0.958_0.499_0
- removed link upper_left_cabinet_1.003_0.958_0.499_0_corpus
- removed link upper_left_cabinet_1.003_0.958_0.499_0_door_0_0
- removed link upper_left_cabinet_1.003_0.958_0.499_1
- removed link upper_left_cabinet_1.003_0.958_0.499_1_corpus
- removed link upper_left_cabinet_1.003_0.958_0.499_1_door_0_0
- removed link upper_left_cabinet_1.003_0.958_0.499_2
- removed link upper_left_cabinet_1.003_0.958_0.499_2_corpus
- removed link upper_left_cabinet_1.003_0.958_0.499_2_door_0_0
- removed link upper_left_cabinet_1.003_0.958_0.499_3
- removed link upper_left_cabinet_1.003_0.958_0.499_3_corpus
- removed link upper_left_cabinet_1.003_0.958_0.499_3_door_0_0
- removed link upper_right_cabinet_1.003_0.958_0.499_0
- removed link upper_right_cabinet_1.003_0.958_0.499_0_corpus
- removed link upper_right_cabinet_1.003_0.958_0.499_0_door_0_0
- removed link upper_right_cabinet_1.003_0.958_0.499_1
- removed link upper_right_cabinet_1.003_0.958_0.499_1_corpus
- removed link upper_right_cabinet_1.003_0.958_0.499_1_door_0_0
- removed link upper_right_cabinet_1.003_0.958_0.499_2
- removed link upper_right_cabinet_1.003_0.958_0.499_2_corpus
- removed link upper_right_cabinet_1.003_0.958_0.499_2_door_0_0
- removed link upper_right_cabinet_1.003_0.958_0.499_3
- removed link upper_right_cabinet_1.003_0.958_0.499_3_corpus
- removed link upper_right_cabinet_1.003_0.958_0.499_3_door_0_0
- added link big_drawer_0.49950000000000006_0.958_0.998_0
- added link big_drawer_0.49950000000000006_0.958_0.998_0_corpus, mass 0.06388902; collision box size=0.02 0.958 0.47950000000000004; collision box size=0.02 0.958 0.47950000000000004
- added link big_drawer_0.49950000000000006_0.958_0.998_0_drawer_0_0, mass 0.09999999999999999; collision box size=0.005 0.8552 0.44950000000000007; collision box size=0.005 0.8552 0.44950000000000007
- added link big_drawer_0.49950000000000006_0.958_0.998_1
- added link big_drawer_0.49950000000000006_0.958_0.998_1_corpus, mass 0.06388902; collision box size=0.02 0.958 0.47950000000000004; collision box size=0.02 0.958 0.47950000000000004
- added link big_drawer_0.49950000000000006_0.958_0.998_1_drawer_0_0, mass 0.09999999999999999; collision box size=0.005 0.8552 0.44950000000000007; collision box size=0.005 0.8552 0.44950000000000007
- added link big_upper_cabinet_2.103_0.958_0.499_3
- added link big_upper_cabinet_2.103_0.958_0.499_3_corpus, mass 0.05906136; collision box size=0.01 0.469 2.0930000000000004; collision box size=0.01 0.469 2.0930000000000004
- added link big_upper_cabinet_2.103_0.958_0.499_3_door_0_0, mass 0.1; collision box size=0.013999999999999999 0.04 0.024; collision box size=0.013999999999999999 0.04 0.024
- added link box, mass 1.2641282767999997; collision box size=0.9480999999999999 0.998 1.3359999999999999; visual box size=0.9480999999999999 0.998 1.3359999999999999
- added link drawer_0.333_0.958_0.998_10
- added link drawer_0.333_0.958_0.998_10_corpus, mass 0.054318599999999995; collision box size=0.02 0.958 0.313; collision box size=0.02 0.958 0.313
- added link drawer_0.333_0.958_0.998_10_drawer_0_0, mass 0.1; collision box size=0.005 0.8552 0.28300000000000003; collision box size=0.005 0.8552 0.28300000000000003
- added link drawer_0.333_0.958_0.998_6
- added link drawer_0.333_0.958_0.998_6_corpus, mass 0.054318599999999995; collision box size=0.02 0.958 0.313; collision box size=0.02 0.958 0.313
- added link drawer_0.333_0.958_0.998_6_drawer_0_0, mass 0.1; collision box size=0.005 0.8552 0.28300000000000003; collision box size=0.005 0.8552 0.28300000000000003
- added link drawer_0.333_0.958_0.998_7
- added link drawer_0.333_0.958_0.998_7_corpus, mass 0.054318599999999995; collision box size=0.02 0.958 0.313; collision box size=0.02 0.958 0.313
- added link drawer_0.333_0.958_0.998_7_drawer_0_0, mass 0.1; collision box size=0.005 0.8552 0.28300000000000003; collision box size=0.005 0.8552 0.28300000000000003
- added link drawer_0.333_0.958_0.998_8
- added link drawer_0.333_0.958_0.998_8_corpus, mass 0.054318599999999995; collision box size=0.02 0.958 0.313; collision box size=0.02 0.958 0.313
- added link drawer_0.333_0.958_0.998_8_drawer_0_0, mass 0.1; collision box size=0.005 0.8552 0.28300000000000003; collision box size=0.005 0.8552 0.28300000000000003
- added link drawer_0.333_0.958_0.998_9
- added link drawer_0.333_0.958_0.998_9_corpus, mass 0.054318599999999995; collision box size=0.02 0.958 0.313; collision box size=0.02 0.958 0.313
- added link drawer_0.333_0.958_0.998_9_drawer_0_0, mass 0.1; collision box size=0.005 0.8552 0.28300000000000003; collision box size=0.005 0.8552 0.28300000000000003
- added link long_drawer
- added link long_drawer_corpus, mass 0.09740943999999999; collision box size=0.02 0.958 0.313; collision box size=0.02 0.958 0.313
- added link long_drawer_drawer_0_0, mass 0.10000000000000005; collision box size=0.0 0.04 0.0; collision box size=0.0 0.04 0.0
- added link lower_left_cabinet_2.103_0.958_0.499_0
- added link lower_left_cabinet_2.103_0.958_0.499_0_corpus, mass 0.10162463999999999; collision box size=0.02 0.958 0.9829999999999999; collision box size=0.02 0.958 0.9829999999999999
- added link lower_left_cabinet_2.103_0.958_0.499_0_door_0_0, mass 0.1; collision box size=0.013999999999999999 0.04 0.024; collision box size=0.013999999999999999 0.04 0.024
- added link lower_left_cabinet_2.103_0.958_0.499_1
- added link lower_left_cabinet_2.103_0.958_0.499_1_corpus, mass 0.10162463999999999; collision box size=0.02 0.958 0.9829999999999999; collision box size=0.02 0.958 0.9829999999999999
- added link lower_left_cabinet_2.103_0.958_0.499_1_door_0_0, mass 0.1; collision box size=0.013999999999999999 0.04 0.024; collision box size=0.013999999999999999 0.04 0.024
- added link lower_left_cabinet_2.103_0.958_0.499_2
- added link lower_left_cabinet_2.103_0.958_0.499_2_corpus, mass 0.10162463999999999; collision box size=0.02 0.958 0.9829999999999999; collision box size=0.02 0.958 0.9829999999999999
- added link lower_left_cabinet_2.103_0.958_0.499_2_door_0_0, mass 0.1; collision box size=0.013999999999999999 0.04 0.024; collision box size=0.013999999999999999 0.04 0.024
- added link lower_left_cabinet_2.103_0.958_0.499_3
- added link lower_left_cabinet_2.103_0.958_0.499_3_corpus, mass 0.10162463999999999; collision box size=0.02 0.958 0.9829999999999999; collision box size=0.02 0.958 0.9829999999999999
- added link lower_left_cabinet_2.103_0.958_0.499_3_door_0_0, mass 0.1; collision box size=0.013999999999999999 0.04 0.024; collision box size=0.013999999999999999 0.04 0.024
- added link lower_left_cabinet_2.103_0.958_0.499_4
- added link lower_left_cabinet_2.103_0.958_0.499_4_corpus, mass 0.10162463999999999; collision box size=0.02 0.958 0.9829999999999999; collision box size=0.02 0.958 0.9829999999999999
- added link lower_left_cabinet_2.103_0.958_0.499_4_door_0_0, mass 0.1; collision box size=0.013999999999999999 0.04 0.024; collision box size=0.013999999999999999 0.04 0.024
- added link lower_left_cabinet_2.103_0.958_0.499_5
- added link lower_left_cabinet_2.103_0.958_0.499_5_corpus, mass 0.10162463999999999; collision box size=0.02 0.958 0.9829999999999999; collision box size=0.02 0.958 0.9829999999999999
- added link lower_left_cabinet_2.103_0.958_0.499_5_door_0_0, mass 0.1; collision box size=0.013999999999999999 0.04 0.024; collision box size=0.013999999999999999 0.04 0.024
- added link lower_left_cabinet_2.103_0.958_0.499_6
- added link lower_left_cabinet_2.103_0.958_0.499_6_corpus, mass 0.10162463999999999; collision box size=0.02 0.958 0.9829999999999999; collision box size=0.02 0.958 0.9829999999999999
- added link lower_left_cabinet_2.103_0.958_0.499_6_door_0_0, mass 0.1; collision box size=0.013999999999999999 0.04 0.024; collision box size=0.013999999999999999 0.04 0.024
- added link lower_right_cabinet_1.003_0.958_0.998_3
- added link lower_right_cabinet_1.003_0.958_0.998_3_corpus, mass 0.10162463999999999; collision box size=0.02 0.958 0.9829999999999999; collision box size=0.02 0.958 0.9829999999999999
- added link lower_right_cabinet_1.003_0.958_0.998_3_door_0_0, mass 0.1; collision box size=0.013999999999999999 0.04 0.024; collision box size=0.013999999999999999 0.04 0.024
- added link lower_right_cabinet_1.003_0.958_0.998_4
- added link lower_right_cabinet_1.003_0.958_0.998_4_corpus, mass 0.10162463999999999; collision box size=0.02 0.958 0.9829999999999999; collision box size=0.02 0.958 0.9829999999999999
- added link lower_right_cabinet_1.003_0.958_0.998_4_door_0_0, mass 0.1; collision box size=0.013999999999999999 0.04 0.024; collision box size=0.013999999999999999 0.04 0.024
- added link lower_right_cabinet_1.003_0.958_0.998_5
- added link lower_right_cabinet_1.003_0.958_0.998_5_corpus, mass 0.10162463999999999; collision box size=0.02 0.958 0.9829999999999999; collision box size=0.02 0.958 0.9829999999999999
- added link lower_right_cabinet_1.003_0.958_0.998_5_door_0_0, mass 0.1; collision box size=0.013999999999999999 0.04 0.024; collision box size=0.013999999999999999 0.04 0.024
- added link upper_left_cabinet_2.103_0.958_0.499_0
- added link upper_left_cabinet_2.103_0.958_0.499_0_corpus, mass 0.05746976000000001; collision box size=0.01 0.469 2.0930000000000004; collision box size=0.01 0.469 2.0930000000000004
- added link upper_left_cabinet_2.103_0.958_0.499_0_door_0_0, mass 0.09999999999999998; collision box size=0.013999999999999999 0.04 0.024; collision box size=0.013999999999999999 0.04 0.024
- added link upper_left_cabinet_2.103_0.958_0.499_1
- added link upper_left_cabinet_2.103_0.958_0.499_1_corpus, mass 0.05746976000000001; collision box size=0.01 0.469 2.0930000000000004; collision box size=0.01 0.469 2.0930000000000004
- added link upper_left_cabinet_2.103_0.958_0.499_1_door_0_0, mass 0.09999999999999998; collision box size=0.013999999999999999 0.04 0.024; collision box size=0.013999999999999999 0.04 0.024
- added link upper_left_cabinet_2.103_0.958_0.499_2
- added link upper_left_cabinet_2.103_0.958_0.499_2_corpus, mass 0.05746976000000001; collision box size=0.01 0.469 2.0930000000000004; collision box size=0.01 0.469 2.0930000000000004
- added link upper_left_cabinet_2.103_0.958_0.499_2_door_0_0, mass 0.09999999999999998; collision box size=0.013999999999999999 0.04 0.024; collision box size=0.013999999999999999 0.04 0.024
- added link upper_right_cabinet_2.103_0.958_0.499_0
- added link upper_right_cabinet_2.103_0.958_0.499_0_corpus, mass 0.05746976000000001; collision box size=0.01 0.469 2.0930000000000004; collision box size=0.01 0.469 2.0930000000000004
- added link upper_right_cabinet_2.103_0.958_0.499_0_door_0_0, mass 0.09999999999999998; collision box size=0.013999999999999999 0.04 0.024; collision box size=0.013999999999999999 0.04 0.024
- added link upper_right_cabinet_2.103_0.958_0.499_1
- added link upper_right_cabinet_2.103_0.958_0.499_1_corpus, mass 0.05746976000000001; collision box size=0.01 0.469 2.0930000000000004; collision box size=0.01 0.469 2.0930000000000004
- added link upper_right_cabinet_2.103_0.958_0.499_1_door_0_0, mass 0.09999999999999998; collision box size=0.013999999999999999 0.04 0.024; collision box size=0.013999999999999999 0.04 0.024
- added link upper_right_cabinet_2.103_0.958_0.499_2
- added link upper_right_cabinet_2.103_0.958_0.499_2_corpus, mass 0.05746976000000001; collision box size=0.01 0.469 2.0930000000000004; collision box size=0.01 0.469 2.0930000000000004
- added link upper_right_cabinet_2.103_0.958_0.499_2_door_0_0, mass 0.09999999999999998; collision box size=0.013999999999999999 0.04 0.024; collision box size=0.013999999999999999 0.04 0.024
- added link upper_right_cabinet_2.103_0.958_0.499_3
- added link upper_right_cabinet_2.103_0.958_0.499_3_corpus, mass 0.05746976000000001; collision box size=0.01 0.469 2.0930000000000004; collision box size=0.01 0.469 2.0930000000000004
- added link upper_right_cabinet_2.103_0.958_0.499_3_door_0_0, mass 0.09999999999999998; collision box size=0.013999999999999999 0.04 0.024; collision box size=0.013999999999999999 0.04 0.024
- link counter_0: mass 0.40235839056000006 -> 0.9416362334399998; geometry collision box size=13.451999999999998 1.0479 0.0668; visual box size=13.451999999999998 1.0479 0.0668
Joints:
- removed joint double_drawer_0.49950000000000006_1.916_0.998_corpus_to_drawer_0_0
- removed joint double_drawer_0.49950000000000006_1.916_0.998_origin_joint
- removed joint double_drawer_0.49950000000000006_1.916_0.998_world_fixed_joint
- removed joint lower_left_cabinet_1.003_0.958_0.998_0_corpus_to_door_0_0
- removed joint lower_left_cabinet_1.003_0.958_0.998_0_origin_joint
- removed joint lower_left_cabinet_1.003_0.958_0.998_0_world_fixed_joint
- removed joint lower_left_cabinet_1.003_0.958_0.998_1_corpus_to_door_0_0
- removed joint lower_left_cabinet_1.003_0.958_0.998_1_origin_joint
- removed joint lower_left_cabinet_1.003_0.958_0.998_1_world_fixed_joint
- removed joint lower_left_cabinet_1.003_0.958_0.998_2_corpus_to_door_0_0
- removed joint lower_left_cabinet_1.003_0.958_0.998_2_origin_joint
- removed joint lower_left_cabinet_1.003_0.958_0.998_2_world_fixed_joint
- removed joint titled_upper_right_cabinet_2.103_0.7056925676241745_0.7056925676241744_0_corpus_to_door_0_0
- removed joint titled_upper_right_cabinet_2.103_0.7056925676241745_0.7056925676241744_0_origin_joint
- removed joint titled_upper_right_cabinet_2.103_0.7056925676241745_0.7056925676241744_0_world_fixed_joint
- removed joint upper_left_cabinet_1.003_0.958_0.499_0_corpus_to_door_0_0
- removed joint upper_left_cabinet_1.003_0.958_0.499_0_origin_joint
- removed joint upper_left_cabinet_1.003_0.958_0.499_0_world_fixed_joint
- removed joint upper_left_cabinet_1.003_0.958_0.499_1_corpus_to_door_0_0
- removed joint upper_left_cabinet_1.003_0.958_0.499_1_origin_joint
- removed joint upper_left_cabinet_1.003_0.958_0.499_1_world_fixed_joint
- removed joint upper_left_cabinet_1.003_0.958_0.499_2_corpus_to_door_0_0
- removed joint upper_left_cabinet_1.003_0.958_0.499_2_origin_joint
- removed joint upper_left_cabinet_1.003_0.958_0.499_2_world_fixed_joint
- removed joint upper_left_cabinet_1.003_0.958_0.499_3_corpus_to_door_0_0
- removed joint upper_left_cabinet_1.003_0.958_0.499_3_origin_joint
- removed joint upper_left_cabinet_1.003_0.958_0.499_3_world_fixed_joint
- removed joint upper_right_cabinet_1.003_0.958_0.499_0_corpus_to_door_0_0
- removed joint upper_right_cabinet_1.003_0.958_0.499_0_origin_joint
- removed joint upper_right_cabinet_1.003_0.958_0.499_0_world_fixed_joint
- removed joint upper_right_cabinet_1.003_0.958_0.499_1_corpus_to_door_0_0
- removed joint upper_right_cabinet_1.003_0.958_0.499_1_origin_joint
- removed joint upper_right_cabinet_1.003_0.958_0.499_1_world_fixed_joint
- removed joint upper_right_cabinet_1.003_0.958_0.499_2_corpus_to_door_0_0
- removed joint upper_right_cabinet_1.003_0.958_0.499_2_origin_joint
- removed joint upper_right_cabinet_1.003_0.958_0.499_2_world_fixed_joint
- removed joint upper_right_cabinet_1.003_0.958_0.499_3_corpus_to_door_0_0
- removed joint upper_right_cabinet_1.003_0.958_0.499_3_origin_joint
- removed joint upper_right_cabinet_1.003_0.958_0.499_3_world_fixed_joint
- added joint big_drawer_0.49950000000000006_0.958_0.998_0_corpus_to_drawer_0_0: type prismatic, parent big_drawer_0.49950000000000006_0.958_0.998_0_corpus, child big_drawer_0.49950000000000006_0.958_0.998_0_drawer_0_0, origin xyz=0.0 -0.479 0.24975 rpy=0.0 -0.0 0.0, axis 0 -1 0, limit lower=0.0 upper=0.79218 effort=1000.0 velocity=1.0
- added joint big_drawer_0.49950000000000006_0.958_0.998_0_origin_joint: type fixed, parent big_drawer_0.49950000000000006_0.958_0.998_0, child big_drawer_0.49950000000000006_0.958_0.998_0_corpus, origin xyz=0.0 0.0 0.0 rpy=0.0 -0.0 0.0
- added joint big_drawer_0.49950000000000006_0.958_0.998_0_world_fixed_joint: type fixed, parent world, child big_drawer_0.49950000000000006_0.958_0.998_0, origin xyz=1.936 -6.726000000000001 -1.003 rpy=0.0 -0.0 -1.5707963267948966
- added joint big_drawer_0.49950000000000006_0.958_0.998_1_corpus_to_drawer_0_0: type prismatic, parent big_drawer_0.49950000000000006_0.958_0.998_1_corpus, child big_drawer_0.49950000000000006_0.958_0.998_1_drawer_0_0, origin xyz=0.0 -0.479 0.24975 rpy=0.0 -0.0 0.0, axis 0 -1 0, limit lower=0.0 upper=0.79218 effort=1000.0 velocity=1.0
- added joint big_drawer_0.49950000000000006_0.958_0.998_1_origin_joint: type fixed, parent big_drawer_0.49950000000000006_0.958_0.998_1, child big_drawer_0.49950000000000006_0.958_0.998_1_corpus, origin xyz=0.0 0.0 0.0 rpy=0.0 -0.0 0.0
- added joint big_drawer_0.49950000000000006_0.958_0.998_1_world_fixed_joint: type fixed, parent world, child big_drawer_0.49950000000000006_0.958_0.998_1, origin xyz=1.936 -7.684000000000001 -1.003 rpy=0.0 -0.0 -1.5707963267948966
- added joint big_upper_cabinet_2.103_0.958_0.499_3_corpus_to_door_0_0: type revolute, parent big_upper_cabinet_2.103_0.958_0.499_3_corpus, child big_upper_cabinet_2.103_0.958_0.499_3_door_0_0, origin xyz=0.498 -0.2495 1.0515000000000003 rpy=0.0 -0.0 0.0, axis 0 0 1, limit lower=0.0 upper=1.5707963267948966 effort=1000.0 velocity=0.1
- added joint big_upper_cabinet_2.103_0.958_0.499_3_origin_joint: type fixed, parent big_upper_cabinet_2.103_0.958_0.499_3, child big_upper_cabinet_2.103_0.958_0.499_3_corpus, origin xyz=0.0 0.0 0.0 rpy=0.0 -0.0 0.0
- added joint big_upper_cabinet_2.103_0.958_0.499_3_world_fixed_joint: type fixed, parent world, child big_upper_cabinet_2.103_0.958_0.499_3, origin xyz=1.936 0.2495 1.2330000000000003 rpy=0.0 -0.0 0.0
- added joint box_world_fixed_joint: type fixed, parent world, child box, origin xyz=1.96095 -13.451999999999995 -0.33499999999999996 rpy=0.0 -0.0 3.141592653589793
- added joint drawer_0.333_0.958_0.998_10_corpus_to_drawer_0_0: type prismatic, parent drawer_0.333_0.958_0.998_10_corpus, child drawer_0.333_0.958_0.998_10_drawer_0_0, origin xyz=0.0 -0.479 0.16649999999999998 rpy=0.0 -0.0 0.0, axis 0 -1 0, limit lower=0.0 upper=0.79218 effort=1000.0 velocity=1.0
- added joint drawer_0.333_0.958_0.998_10_origin_joint: type fixed, parent drawer_0.333_0.958_0.998_10, child drawer_0.333_0.958_0.998_10_corpus, origin xyz=0.0 0.0 0.0 rpy=0.0 -0.0 0.0
- added joint drawer_0.333_0.958_0.998_10_world_fixed_joint: type fixed, parent world, child drawer_0.333_0.958_0.998_10, origin xyz=1.936 -12.473999999999995 0.0 rpy=0.0 -0.0 -1.5707963267948966
- added joint drawer_0.333_0.958_0.998_6_corpus_to_drawer_0_0: type prismatic, parent drawer_0.333_0.958_0.998_6_corpus, child drawer_0.333_0.958_0.998_6_drawer_0_0, origin xyz=0.0 -0.479 0.16649999999999998 rpy=0.0 -0.0 0.0, axis 0 -1 0, limit lower=0.0 upper=0.79218 effort=1000.0 velocity=1.0
- added joint drawer_0.333_0.958_0.998_6_origin_joint: type fixed, parent drawer_0.333_0.958_0.998_6, child drawer_0.333_0.958_0.998_6_corpus, origin xyz=0.0 0.0 0.0 rpy=0.0 -0.0 0.0
- added joint drawer_0.333_0.958_0.998_6_world_fixed_joint: type fixed, parent world, child drawer_0.333_0.958_0.998_6, origin xyz=1.936 -8.642000000000001 0.0 rpy=0.0 -0.0 -1.5707963267948966
- added joint drawer_0.333_0.958_0.998_7_corpus_to_drawer_0_0: type prismatic, parent drawer_0.333_0.958_0.998_7_corpus, child drawer_0.333_0.958_0.998_7_drawer_0_0, origin xyz=0.0 -0.479 0.16649999999999998 rpy=0.0 -0.0 0.0, axis 0 -1 0, limit lower=0.0 upper=0.79218 effort=1000.0 velocity=1.0
- added joint drawer_0.333_0.958_0.998_7_origin_joint: type fixed, parent drawer_0.333_0.958_0.998_7, child drawer_0.333_0.958_0.998_7_corpus, origin xyz=0.0 0.0 0.0 rpy=0.0 -0.0 0.0
- added joint drawer_0.333_0.958_0.998_7_world_fixed_joint: type fixed, parent world, child drawer_0.333_0.958_0.998_7, origin xyz=1.936 -9.6 0.0 rpy=0.0 -0.0 -1.5707963267948966
- added joint drawer_0.333_0.958_0.998_8_corpus_to_drawer_0_0: type prismatic, parent drawer_0.333_0.958_0.998_8_corpus, child drawer_0.333_0.958_0.998_8_drawer_0_0, origin xyz=0.0 -0.479 0.16649999999999998 rpy=0.0 -0.0 0.0, axis 0 -1 0, limit lower=0.0 upper=0.79218 effort=1000.0 velocity=1.0
- added joint drawer_0.333_0.958_0.998_8_origin_joint: type fixed, parent drawer_0.333_0.958_0.998_8, child drawer_0.333_0.958_0.998_8_corpus, origin xyz=0.0 0.0 0.0 rpy=0.0 -0.0 0.0
- added joint drawer_0.333_0.958_0.998_8_world_fixed_joint: type fixed, parent world, child drawer_0.333_0.958_0.998_8, origin xyz=1.936 -10.557999999999998 0.0 rpy=0.0 -0.0 -1.5707963267948966
- added joint drawer_0.333_0.958_0.998_9_corpus_to_drawer_0_0: type prismatic, parent drawer_0.333_0.958_0.998_9_corpus, child drawer_0.333_0.958_0.998_9_drawer_0_0, origin xyz=0.0 -0.479 0.16649999999999998 rpy=0.0 -0.0 0.0, axis 0 -1 0, limit lower=0.0 upper=0.79218 effort=1000.0 velocity=1.0
- added joint drawer_0.333_0.958_0.998_9_origin_joint: type fixed, parent drawer_0.333_0.958_0.998_9, child drawer_0.333_0.958_0.998_9_corpus, origin xyz=0.0 0.0 0.0 rpy=0.0 -0.0 0.0
- added joint drawer_0.333_0.958_0.998_9_world_fixed_joint: type fixed, parent world, child drawer_0.333_0.958_0.998_9, origin xyz=1.936 -11.515999999999996 0.0 rpy=0.0 -0.0 -1.5707963267948966
- added joint long_drawer_corpus_to_drawer_0_0: type prismatic, parent long_drawer_corpus, child long_drawer_drawer_0_0, origin xyz=0.0 -0.479 0.16649999999999998 rpy=0.0 -0.0 0.0, axis 0 -1 0, limit lower=0.0 upper=0.79218 effort=1000.0 velocity=1.0
- added joint long_drawer_origin_joint: type fixed, parent long_drawer, child long_drawer_corpus, origin xyz=0.0 0.0 0.0 rpy=0.0 -0.0 0.0
- added joint long_drawer_world_fixed_joint: type fixed, parent world, child long_drawer, origin xyz=1.936 -3.373 0.0 rpy=0.0 -0.0 -1.5707963267948966
- added joint lower_left_cabinet_2.103_0.958_0.499_0_corpus_to_door_0_0: type revolute, parent lower_left_cabinet_2.103_0.958_0.499_0_corpus, child lower_left_cabinet_2.103_0.958_0.499_0_door_0_0, origin xyz=0.477 -0.499 0.5015 rpy=0.0 -0.0 0.0, axis 0 0 1, limit lower=0.0 upper=1.5707963267948966 effort=1000.0 velocity=0.1
- added joint lower_left_cabinet_2.103_0.958_0.499_0_origin_joint: type fixed, parent lower_left_cabinet_2.103_0.958_0.499_0, child lower_left_cabinet_2.103_0.958_0.499_0_corpus, origin xyz=0.0 0.0 0.0 rpy=0.0 -0.0 0.0
- added joint lower_left_cabinet_2.103_0.958_0.499_0_world_fixed_joint: type fixed, parent world, child lower_left_cabinet_2.103_0.958_0.499_0, origin xyz=0.958 0.0 -1.003 rpy=0.0 -0.0 0.0
- added joint lower_left_cabinet_2.103_0.958_0.499_1_corpus_to_door_0_0: type revolute, parent lower_left_cabinet_2.103_0.958_0.499_1_corpus, child lower_left_cabinet_2.103_0.958_0.499_1_door_0_0, origin xyz=0.477 -0.499 0.5015 rpy=0.0 -0.0 0.0, axis 0 0 1, limit lower=0.0 upper=1.5707963267948966 effort=1000.0 velocity=0.1
- added joint lower_left_cabinet_2.103_0.958_0.499_1_origin_joint: type fixed, parent lower_left_cabinet_2.103_0.958_0.499_1, child lower_left_cabinet_2.103_0.958_0.499_1_corpus, origin xyz=0.0 0.0 0.0 rpy=0.0 -0.0 0.0
- added joint lower_left_cabinet_2.103_0.958_0.499_1_world_fixed_joint: type fixed, parent world, child lower_left_cabinet_2.103_0.958_0.499_1, origin xyz=1.936 -1.936 -1.003 rpy=0.0 -0.0 -1.5707963267948966
- added joint lower_left_cabinet_2.103_0.958_0.499_2_corpus_to_door_0_0: type revolute, parent lower_left_cabinet_2.103_0.958_0.499_2_corpus, child lower_left_cabinet_2.103_0.958_0.499_2_door_0_0, origin xyz=0.477 -0.499 0.5015 rpy=0.0 -0.0 0.0, axis 0 0 1, limit lower=0.0 upper=1.5707963267948966 effort=1000.0 velocity=0.1
- added joint lower_left_cabinet_2.103_0.958_0.499_2_origin_joint: type fixed, parent lower_left_cabinet_2.103_0.958_0.499_2, child lower_left_cabinet_2.103_0.958_0.499_2_corpus, origin xyz=0.0 0.0 0.0 rpy=0.0 -0.0 0.0
- added joint lower_left_cabinet_2.103_0.958_0.499_2_world_fixed_joint: type fixed, parent world, child lower_left_cabinet_2.103_0.958_0.499_2, origin xyz=1.936 -5.768000000000001 -1.003 rpy=0.0 -0.0 -1.5707963267948966
- added joint lower_left_cabinet_2.103_0.958_0.499_3_corpus_to_door_0_0: type revolute, parent lower_left_cabinet_2.103_0.958_0.499_3_corpus, child lower_left_cabinet_2.103_0.958_0.499_3_door_0_0, origin xyz=0.477 -0.499 0.5015 rpy=0.0 -0.0 0.0, axis 0 0 1, limit lower=0.0 upper=1.5707963267948966 effort=1000.0 velocity=0.1
- added joint lower_left_cabinet_2.103_0.958_0.499_3_origin_joint: type fixed, parent lower_left_cabinet_2.103_0.958_0.499_3, child lower_left_cabinet_2.103_0.958_0.499_3_corpus, origin xyz=0.0 0.0 0.0 rpy=0.0 -0.0 0.0
- added joint lower_left_cabinet_2.103_0.958_0.499_3_world_fixed_joint: type fixed, parent world, child lower_left_cabinet_2.103_0.958_0.499_3, origin xyz=1.936 -9.6 -1.003 rpy=0.0 -0.0 -1.5707963267948966
- added joint lower_left_cabinet_2.103_0.958_0.499_4_corpus_to_door_0_0: type revolute, parent lower_left_cabinet_2.103_0.958_0.499_4_corpus, child lower_left_cabinet_2.103_0.958_0.499_4_door_0_0, origin xyz=0.477 -0.499 0.5015 rpy=0.0 -0.0 0.0, axis 0 0 1, limit lower=0.0 upper=1.5707963267948966 effort=1000.0 velocity=0.1
- added joint lower_left_cabinet_2.103_0.958_0.499_4_origin_joint: type fixed, parent lower_left_cabinet_2.103_0.958_0.499_4, child lower_left_cabinet_2.103_0.958_0.499_4_corpus, origin xyz=0.0 0.0 0.0 rpy=0.0 -0.0 0.0
- added joint lower_left_cabinet_2.103_0.958_0.499_4_world_fixed_joint: type fixed, parent world, child lower_left_cabinet_2.103_0.958_0.499_4, origin xyz=1.936 -11.515999999999996 -1.003 rpy=0.0 -0.0 -1.5707963267948966
- added joint lower_left_cabinet_2.103_0.958_0.499_5_corpus_to_door_0_0: type revolute, parent lower_left_cabinet_2.103_0.958_0.499_5_corpus, child lower_left_cabinet_2.103_0.958_0.499_5_door_0_0, origin xyz=0.477 -0.499 0.5015 rpy=0.0 -0.0 0.0, axis 0 0 1, limit lower=0.0 upper=1.5707963267948966 effort=1000.0 velocity=0.1
- added joint lower_left_cabinet_2.103_0.958_0.499_5_origin_joint: type fixed, parent lower_left_cabinet_2.103_0.958_0.499_5, child lower_left_cabinet_2.103_0.958_0.499_5_corpus, origin xyz=0.0 0.0 0.0 rpy=0.0 -0.0 0.0
- added joint lower_left_cabinet_2.103_0.958_0.499_5_world_fixed_joint: type fixed, parent world, child lower_left_cabinet_2.103_0.958_0.499_5, origin xyz=1.936 -3.8520000000000003 -1.003 rpy=0.0 -0.0 -1.5707963267948966
- added joint lower_left_cabinet_2.103_0.958_0.499_6_corpus_to_door_0_0: type revolute, parent lower_left_cabinet_2.103_0.958_0.499_6_corpus, child lower_left_cabinet_2.103_0.958_0.499_6_door_0_0, origin xyz=0.477 -0.499 0.5015 rpy=0.0 -0.0 0.0, axis 0 0 1, limit lower=0.0 upper=1.5707963267948966 effort=1000.0 velocity=0.1
- added joint lower_left_cabinet_2.103_0.958_0.499_6_origin_joint: type fixed, parent lower_left_cabinet_2.103_0.958_0.499_6, child lower_left_cabinet_2.103_0.958_0.499_6_corpus, origin xyz=0.0 0.0 0.0 rpy=0.0 -0.0 0.0
- added joint lower_left_cabinet_2.103_0.958_0.499_6_world_fixed_joint: type fixed, parent world, child lower_left_cabinet_2.103_0.958_0.499_6, origin xyz=1.936 -12.473999999999995 -1.003 rpy=0.0 -0.0 -1.5707963267948966
- added joint lower_right_cabinet_1.003_0.958_0.998_3_corpus_to_door_0_0: type revolute, parent lower_right_cabinet_1.003_0.958_0.998_3_corpus, child lower_right_cabinet_1.003_0.958_0.998_3_door_0_0, origin xyz=-0.477 -0.499 0.5015 rpy=0.0 -0.0 0.0, axis 0 0 -1, limit lower=0.0 upper=1.5707963267948966 effort=1000.0 velocity=0.1
- added joint lower_right_cabinet_1.003_0.958_0.998_3_origin_joint: type fixed, parent lower_right_cabinet_1.003_0.958_0.998_3, child lower_right_cabinet_1.003_0.958_0.998_3_corpus, origin xyz=0.0 0.0 0.0 rpy=0.0 -0.0 0.0
- added joint lower_right_cabinet_1.003_0.958_0.998_3_world_fixed_joint: type fixed, parent world, child lower_right_cabinet_1.003_0.958_0.998_3, origin xyz=1.936 -8.642000000000001 -1.003 rpy=0.0 -0.0 -1.5707963267948966
- added joint lower_right_cabinet_1.003_0.958_0.998_4_corpus_to_door_0_0: type revolute, parent lower_right_cabinet_1.003_0.958_0.998_4_corpus, child lower_right_cabinet_1.003_0.958_0.998_4_door_0_0, origin xyz=-0.477 -0.499 0.5015 rpy=0.0 -0.0 0.0, axis 0 0 -1, limit lower=0.0 upper=1.5707963267948966 effort=1000.0 velocity=0.1
- added joint lower_right_cabinet_1.003_0.958_0.998_4_origin_joint: type fixed, parent lower_right_cabinet_1.003_0.958_0.998_4, child lower_right_cabinet_1.003_0.958_0.998_4_corpus, origin xyz=0.0 0.0 0.0 rpy=0.0 -0.0 0.0
- added joint lower_right_cabinet_1.003_0.958_0.998_4_world_fixed_joint: type fixed, parent world, child lower_right_cabinet_1.003_0.958_0.998_4, origin xyz=1.936 -10.557999999999998 -1.003 rpy=0.0 -0.0 -1.5707963267948966
- added joint lower_right_cabinet_1.003_0.958_0.998_5_corpus_to_door_0_0: type revolute, parent lower_right_cabinet_1.003_0.958_0.998_5_corpus, child lower_right_cabinet_1.003_0.958_0.998_5_door_0_0, origin xyz=-0.477 -0.499 0.5015 rpy=0.0 -0.0 0.0, axis 0 0 -1, limit lower=0.0 upper=1.5707963267948966 effort=1000.0 velocity=0.1
- added joint lower_right_cabinet_1.003_0.958_0.998_5_origin_joint: type fixed, parent lower_right_cabinet_1.003_0.958_0.998_5, child lower_right_cabinet_1.003_0.958_0.998_5_corpus, origin xyz=0.0 0.0 0.0 rpy=0.0 -0.0 0.0
- added joint lower_right_cabinet_1.003_0.958_0.998_5_world_fixed_joint: type fixed, parent world, child lower_right_cabinet_1.003_0.958_0.998_5, origin xyz=1.936 -2.894 -1.003 rpy=0.0 -0.0 -1.5707963267948966
- added joint upper_left_cabinet_2.103_0.958_0.499_0_corpus_to_door_0_0: type revolute, parent upper_left_cabinet_2.103_0.958_0.499_0_corpus, child upper_left_cabinet_2.103_0.958_0.499_0_door_0_0, origin xyz=0.478 -0.2495 1.0515000000000003 rpy=0.0 -0.0 0.0, axis 0 0 1, limit lower=0.0 upper=1.5707963267948966 effort=1000.0 velocity=0.1
- added joint upper_left_cabinet_2.103_0.958_0.499_0_origin_joint: type fixed, parent upper_left_cabinet_2.103_0.958_0.499_0, child upper_left_cabinet_2.103_0.958_0.499_0_corpus, origin xyz=0.0 0.0 0.0 rpy=0.0 -0.0 0.0
- added joint upper_left_cabinet_2.103_0.958_0.499_0_world_fixed_joint: type fixed, parent world, child upper_left_cabinet_2.103_0.958_0.499_0, origin xyz=0.039999999999999925 -13.7015 1.2330000000000003 rpy=0.0 -0.0 3.141592653589793
- added joint upper_left_cabinet_2.103_0.958_0.499_1_corpus_to_door_0_0: type revolute, parent upper_left_cabinet_2.103_0.958_0.499_1_corpus, child upper_left_cabinet_2.103_0.958_0.499_1_door_0_0, origin xyz=0.478 -0.2495 1.0515000000000003 rpy=0.0 -0.0 0.0, axis 0 0 1, limit lower=0.0 upper=1.5707963267948966 effort=1000.0 velocity=0.1
- added joint upper_left_cabinet_2.103_0.958_0.499_1_origin_joint: type fixed, parent upper_left_cabinet_2.103_0.958_0.499_1, child upper_left_cabinet_2.103_0.958_0.499_1_corpus, origin xyz=0.0 0.0 0.0 rpy=0.0 -0.0 0.0
- added joint upper_left_cabinet_2.103_0.958_0.499_1_world_fixed_joint: type fixed, parent world, child upper_left_cabinet_2.103_0.958_0.499_1, origin xyz=-1.876 -13.701500000000003 1.2330000000000003 rpy=0.0 -0.0 3.141592653589793
- added joint upper_left_cabinet_2.103_0.958_0.499_2_corpus_to_door_0_0: type revolute, parent upper_left_cabinet_2.103_0.958_0.499_2_corpus, child upper_left_cabinet_2.103_0.958_0.499_2_door_0_0, origin xyz=0.478 -0.2495 1.0515000000000003 rpy=0.0 -0.0 0.0, axis 0 0 1, limit lower=0.0 upper=1.5707963267948966 effort=1000.0 velocity=0.1
- added joint upper_left_cabinet_2.103_0.958_0.499_2_origin_joint: type fixed, parent upper_left_cabinet_2.103_0.958_0.499_2, child upper_left_cabinet_2.103_0.958_0.499_2_corpus, origin xyz=0.0 0.0 0.0 rpy=0.0 -0.0 0.0
- added joint upper_left_cabinet_2.103_0.958_0.499_2_world_fixed_joint: type fixed, parent world, child upper_left_cabinet_2.103_0.958_0.499_2, origin xyz=0.958 0.2495 1.2330000000000003 rpy=0.0 -0.0 0.0
- added joint upper_right_cabinet_2.103_0.958_0.499_0_corpus_to_door_0_0: type revolute, parent upper_right_cabinet_2.103_0.958_0.499_0_corpus, child upper_right_cabinet_2.103_0.958_0.499_0_door_0_0, origin xyz=-0.478 -0.2495 1.0515000000000003 rpy=0.0 -0.0 0.0, axis 0 0 -1, limit lower=0.0 upper=1.5707963267948966 effort=1000.0 velocity=0.1
- added joint upper_right_cabinet_2.103_0.958_0.499_0_origin_joint: type fixed, parent upper_right_cabinet_2.103_0.958_0.499_0, child upper_right_cabinet_2.103_0.958_0.499_0_corpus, origin xyz=0.0 0.0 0.0 rpy=0.0 -0.0 0.0
- added joint upper_right_cabinet_2.103_0.958_0.499_0_world_fixed_joint: type fixed, parent world, child upper_right_cabinet_2.103_0.958_0.499_0, origin xyz=1.956 -13.701499999999996 1.233 rpy=0.0 -0.0 3.141592653589793
- added joint upper_right_cabinet_2.103_0.958_0.499_1_corpus_to_door_0_0: type revolute, parent upper_right_cabinet_2.103_0.958_0.499_1_corpus, child upper_right_cabinet_2.103_0.958_0.499_1_door_0_0, origin xyz=-0.478 -0.2495 1.0515000000000003 rpy=0.0 -0.0 0.0, axis 0 0 -1, limit lower=0.0 upper=1.5707963267948966 effort=1000.0 velocity=0.1
- added joint upper_right_cabinet_2.103_0.958_0.499_1_origin_joint: type fixed, parent upper_right_cabinet_2.103_0.958_0.499_1, child upper_right_cabinet_2.103_0.958_0.499_1_corpus, origin xyz=0.0 0.0 0.0 rpy=0.0 -0.0 0.0
- added joint upper_right_cabinet_2.103_0.958_0.499_1_world_fixed_joint: type fixed, parent world, child upper_right_cabinet_2.103_0.958_0.499_1, origin xyz=0.9979999999999999 -13.701499999999998 1.2330000000000003 rpy=0.0 -0.0 3.141592653589793
- added joint upper_right_cabinet_2.103_0.958_0.499_2_corpus_to_door_0_0: type revolute, parent upper_right_cabinet_2.103_0.958_0.499_2_corpus, child upper_right_cabinet_2.103_0.958_0.499_2_door_0_0, origin xyz=-0.478 -0.2495 1.0515000000000003 rpy=0.0 -0.0 0.0, axis 0 0 -1, limit lower=0.0 upper=1.5707963267948966 effort=1000.0 velocity=0.1
- added joint upper_right_cabinet_2.103_0.958_0.499_2_origin_joint: type fixed, parent upper_right_cabinet_2.103_0.958_0.499_2, child upper_right_cabinet_2.103_0.958_0.499_2_corpus, origin xyz=0.0 0.0 0.0 rpy=0.0 -0.0 0.0
- added joint upper_right_cabinet_2.103_0.958_0.499_2_world_fixed_joint: type fixed, parent world, child upper_right_cabinet_2.103_0.958_0.499_2, origin xyz=-0.918 -13.701500000000001 1.2330000000000003 rpy=0.0 -0.0 3.141592653589793
- added joint upper_right_cabinet_2.103_0.958_0.499_3_corpus_to_door_0_0: type revolute, parent upper_right_cabinet_2.103_0.958_0.499_3_corpus, child upper_right_cabinet_2.103_0.958_0.499_3_door_0_0, origin xyz=-0.478 -0.2495 1.0515000000000003 rpy=0.0 -0.0 0.0, axis 0 0 -1, limit lower=0.0 upper=1.5707963267948966 effort=1000.0 velocity=0.1
- added joint upper_right_cabinet_2.103_0.958_0.499_3_origin_joint: type fixed, parent upper_right_cabinet_2.103_0.958_0.499_3, child upper_right_cabinet_2.103_0.958_0.499_3_corpus, origin xyz=0.0 0.0 0.0 rpy=0.0 -0.0 0.0
- added joint upper_right_cabinet_2.103_0.958_0.499_3_world_fixed_joint: type fixed, parent world, child upper_right_cabinet_2.103_0.958_0.499_3, origin xyz=0.0 0.2495 1.233 rpy=0.0 -0.0 0.0
- joint counter_0_world_fixed_joint: origin xyz=0.47900000000000054 -0.024950000000000028 0.3664 rpy=0.0 -0.0 0.0 -> xyz=1.91105 -7.224999999999999 0.3664 rpy=0.0 -0.0 -1.5707963267948966
- joint counter_1_world_fixed_joint: origin xyz=3.82705 -0.9580000000000002 0.3664 rpy=0.0 -0.0 -1.5707963267948966 -> xyz=0.9779999999999999 -0.024950000000000028 0.3664 rpy=0.0 -0.0 0.0
- joint drawer_0.333_0.958_0.998_2_world_fixed_joint: origin xyz=1.916 0.0 0.0 rpy=0.0 -0.0 0.0 -> xyz=1.936 -0.9779999999999999 0.0 rpy=0.0 -0.0 -1.5707963267948966
- joint drawer_0.333_0.958_0.998_3_world_fixed_joint: origin xyz=2.874 0.0 0.0 rpy=0.0 -0.0 0.0 -> xyz=1.936 -1.936 0.0 rpy=0.0 -0.0 -1.5707963267948966
- joint drawer_0.333_0.958_0.998_4_world_fixed_joint: origin xyz=3.8520000000000003 -0.9779999999999999 0.0 rpy=0.0 -0.0 -1.5707963267948966 -> xyz=1.936 -4.8100000000000005 0.0 rpy=0.0 -0.0 -1.5707963267948966
- joint drawer_0.333_0.958_0.998_5_world_fixed_joint: origin xyz=3.852 -1.936 0.0 rpy=0.0 -0.0 -1.5707963267948966 -> xyz=1.936 -5.768000000000001 0.0 rpy=0.0 -0.0 -1.5707963267948966
- joint lower_right_cabinet_1.003_0.958_0.998_1_world_fixed_joint: origin xyz=1.916 0.0 -1.003 rpy=0.0 -0.0 0.0 -> xyz=1.936 -0.9779999999999999 -1.003 rpy=0.0 -0.0 -1.5707963267948966
- joint lower_right_cabinet_1.003_0.958_0.998_2_world_fixed_joint: origin xyz=3.852 -0.9779999999999999 -1.003 rpy=0.0 -0.0 -1.5707963267948966 -> xyz=1.936 -4.8100000000000005 -1.003 rpy=0.0 -0.0 -1.5707963267948966
- joint microwave_world_fixed_joint: origin xyz=-1.4369999999999998 0.02065165999999999 -0.5034999999999998 rpy=0.0 -0.0 0.0 -> xyz=1.9566516600000001 -7.205000000000001 -0.5034999999999998 rpy=0.0 -0.0 -1.5707963267948966
- joint refrigerator_world_fixed_joint: origin xyz=-3.3529999999999998 0.0 -1.003 rpy=0.0 -0.0 0.0 -> xyz=-1.4369999999999998 0.0 -1.003 rpy=0.0 -0.0 0.0
